Commit message: Changed the URDF for the inspection cell, made every object in space relative to the table and changed the origin on the table.

File: inspection_cell_description/urdf/inspection_cell_macro.xacro (robot description, xacro)
@@ -519,5 +519,5 @@
     </joint>
     <joint name="${tf_prefix}ur5e_mount_to_table" type="fixed">
-      <origin xyz="0 0 0" rpy="0 0 0"/>
+      <origin xyz="-1.4732 -0.6096 0" rpy="0 0 0"/>
       <parent link="${tf_prefix}ur5e_mount_link"/>
       <child link="${tf_prefix}table_link"/>
@@ -527,5 +527,5 @@
       <parent link="${tf_prefix}turntable_base_link"/>
       <child link="${tf_prefix}ur5e_mount_link"/>
-      <origin xyz="0.97035 0 0" rpy="0 0 0"/>
+      <origin xyz="0.9906 0 0" rpy="0 0 0"/>
     </joint>
     <!-- UR5e Base - Mounted on mount block -->

Commit message: WIP

File: inspection_cell_description/urdf/inspection_cell_macro.xacro (robot description, xacro)
@@ -128,5 +128,5 @@
       </visual>
       <collision>
-        <origin xyz="0 0 -0.4515" rpy="0 0 0"/>
+        <origin xyz="-1.2192 -0.762 -0.4515" rpy="0 0 0"/>
         <geometry>
           <box size="2.4384 1.524 0.903"/>

Commit message: WIP...

File: inspection_cell_description/urdf/inspection_cell_macro.xacro (robot description, xacro)
@@ -128,5 +128,5 @@
       </visual>
       <collision>
-        <origin xyz="-1.2192 -0.762 -0.4515" rpy="0 0 0"/>
+        <origin xyz="1.2192 0.762 -0.4515" rpy="0 0 0"/>
         <geometry>
           <box size="2.4384 1.524 0.903"/>

Commit message: Changed the orientation of the eoat_camera_frame, added a service for triggering the moveit_py trajectory. All of it working in sim and on physical hardware.

File: inspection_cell_description/urdf/inspection_cell_macro.xacro (robot description, xacro)
@@ -686,5 +686,5 @@
       <parent link="${tf_prefix}eoat_base_link"/>
       <child link="${tf_prefix}eoat_camera_link"/>
-      <origin xyz="0 0 0.125" rpy="${radians(90)} ${radians(180)} ${radians(-90)}"/>
+      <origin xyz="0 0 0.125" rpy="${radians(90)} ${radians(0)} ${radians(-90)}"/>
     </joint>
     <!-- ================================================================ -->
