Commit message: Changed the collision for disc link.

File: inspection_cell_description/urdf/inspection_cell.urdf (robot description, URDF)
Before this commit: robot inspection_cell, 22 links, 22 joints
Joints:
- joint base_joint: child turntable_disc_link -> turntable_base_link
- joint turntable_disc_joint: child turntable_base_link -> turntable_disc_link; origin xyz=0 0 0 rpy=0 0 0 -> xyz=0 0 0.1015 rpy=0 0 0; parent turntable_disc_link -> turntable_base_link

File: inspection_cell_description/urdf/inspection_cell_macro.xacro (robot description, xacro)
@@ -147,5 +147,5 @@
       </visual>
       <collision>
-        <origin xyz="0 0 0.1015" rpy="0 0 0"/>
+        <origin xyz="0 0 0" rpy="0 0 0"/>
         <geometry>
           <cylinder length="0.008" radius="0.084"/>

Commit message: Almost correct URDF. But still the visualization is incorrect.

File: inspection_cell_description/urdf/inspection_cell.urdf (robot description, URDF)
Before this commit: robot inspection_cell, 22 links, 22 joints
Links:
- link ur5e_mount_link: mass 5.0 -> None
Joints:
- removed joint table_to_base
- added joint disc_to_base: type fixed, parent turntable_disc_link, child turntable_base_link, origin xyz=0 0 -0.1015 rpy=0 0 0
- joint base_joint: child turntable_base_link -> base_link; origin xyz=-0.76835 0 0 rpy=0 0 0 -> xyz=0 0 0 rpy=0 0 0; parent base_link -> world
- joint base_to_mount: origin xyz=0.2032 0 0.057150 rpy=0 0 0 -> xyz=0.97035 0 0 rpy=0 0 0; parent base_link -> turntable_base_link
- joint mount_to_ur5e: origin xyz=0 0 0.057150 rpy=0 0 0 -> xyz=0 0 0.1143 rpy=0 0 0
- joint table_joint: parent world -> base_link
- joint turntable_disc_joint: origin xyz=0 0 0.1015 rpy=0 0 0 -> xyz=-0.76835 0 0.1015 rpy=0 0 0; parent turntable_base_link -> base_link

File: inspection_cell_description/urdf/inspection_cell_macro.xacro (robot description, xacro)
@@ -3,5 +3,5 @@
   <!--
     Inspection Cell xacro macro - UNIFIED VERSION
-    Kinematic Chain: World → table_link → base_link → turntable_disc_link → turntable_base_link → ur5e_mount_link → ur5e_base_link → ... → eoat_camera_link
+    NEW Kinematic Chain: World → base_link → (table_link | turntable_disc_link → turntable_base_link → ur5e_mount_link → ur_base_link → ... → eoat_camera_link)
   -->
   <!-- Include required dependencies -->
@@ -120,4 +120,6 @@
     <!-- LINK DEFINITIONS -->
     <!-- ================================================================ -->
+    <!-- Base Link - Now the root of our kinematic chain -->
+    <link name="base_link"/>
     <!-- Table Link - 8ft x 5ft x 36in table with top center at (0,0,0) -->
     <link name="${tf_prefix}table_link">
@@ -131,10 +133,12 @@
       <collision>
         <origin xyz="0 0 -0.4572" rpy="0 0 0"/>
-        <geometry>
+        <!-- <geometry>
           <box size="2.4384 1.524 0.9144"/>
-        </geometry>
-      </collision>
-    </link>
-    <link name="base_link"/>
+        </geometry> -->
+        <geometry>
+          <mesh filename="package://inspection_cell_description/meshes/collision/table.stl"/>
+        </geometry>
+      </collision>
+    </link>
     <!-- Turntable Disc Link -->
     <link name="${tf_prefix}turntable_disc_link">
@@ -183,8 +187,8 @@
       </inertial>
     </link>
-    <!-- UR5e Mount Block Link - 7" x 7" x 4.5" -->
+    <!-- UR5e Mount Block Link - 7" x 7" x 4.5" - FRAME AT BASE OF BLOCK -->
     <link name="${tf_prefix}ur5e_mount_link">
       <visual>
-        <origin xyz="0 0 0" rpy="0 0 0"/>
+        <origin xyz="0 0 0.05715" rpy="0 0 0"/>
         <geometry>
           <box size="0.1778 0.1778 0.1143"/>
@@ -193,16 +197,9 @@
       </visual>
       <collision>
-        <origin xyz="0 0 0" rpy="0 0 0"/>
+        <origin xyz="0 0 0.05715" rpy="0 0 0"/>
         <geometry>
           <box size="0.1778 0.1778 0.1143"/>
         </geometry>
       </collision>
-      <inertial>
-        <origin xyz="0 0 0" rpy="0 0 0"/>
-        <mass value="5.0"/>
-        <inertia
-          ixx="0.01" ixy="0.0" ixz="0.0"
-          iyy="0.01" iyz="0.0" izz="0.01" />
-      </inertial>
     </link>
     <!-- ================================================================ -->
@@ -389,5 +386,5 @@
             ixz="${wrist_3_inertia_ixz}"
             iyy="${wrist_3_inertia_iyy}"
-            iyz="${wrist_3_inertia_ixz}"
+            iyz="${wrist_3_inertia_iyz}"
             izz="${wrist_3_inertia_izz}"
         />
@@ -478,29 +475,24 @@
     </link>
     <!-- ================================================================ -->
-    <!-- UNIFIED KINEMATIC CHAIN JOINTS -->
-    <!-- ================================================================ -->
-    <!-- JOINT: Connect parent (world) to table - table positioned so top is at (0,0,0) -->
+    <!-- NEW UNIFIED KINEMATIC CHAIN JOINTS -->
+    <!-- ================================================================ -->
+    <!-- JOINT: Connect parent (world) directly to base_link -->
+    <joint name="${tf_prefix}base_joint" type="fixed">
+      <origin xyz="0 0 0" rpy="0 0 0"/>
+      <parent link="${parent}"/>
+      <child link="base_link"/>
+    </joint>
+    <!-- BRANCH 1: Connect base_link to table_link -->
     <joint name="${tf_prefix}table_joint" type="fixed">
       <origin xyz="0 0 0" rpy="0 0 0"/>
-      <parent link="${parent}"/>
+      <parent link="base_link"/>
       <child link="${tf_prefix}table_link"/>
     </joint>
-    <!-- JOINT: Connect table to base_link (at table surface center, which is (0,0,0)) -->
-    <joint name="${tf_prefix}table_to_base" type="fixed">
-      <origin xyz="0 0 0" rpy="0 0 0"/>
-      <parent link="${tf_prefix}table_link"/>
-      <child link="base_link"/>
-    </joint>
-    <!-- JOINT: Connect base_link to turntable disc (30.25 inches left of center) -->
-    <joint name="${tf_prefix}base_joint" type="fixed">
-      <origin xyz="-0.76835 0 0" rpy="0 0 0"/>
+    <!-- BRANCH 2: MAIN KINEMATIC CHAIN -->
+    <!-- JOINT 1: Turntable disc rotation (DOF 1) - Connect base_link to turntable_disc_link -->
+    <joint name="${tf_prefix}turntable_disc_joint" type="revolute">
       <parent link="base_link"/>
-      <child link="${tf_prefix}turntable_base_link"/>
-    </joint>
-    <!-- JOINT 1: Turntable disc rotation (DOF 1) -->
-    <joint name="${tf_prefix}turntable_disc_joint" type="revolute">
-      <parent link="${tf_prefix}turntable_base_link"/>
       <child link="${tf_prefix}turntable_disc_link"/>
-      <origin xyz="0 0 0.1015" rpy="0 0 0"/>
+      <origin xyz="-0.76835 0 0.1015" rpy="0 0 0"/>
       <axis xyz="0 0 1"/>
       <limit
@@ -518,13 +510,19 @@
       <dynamics damping="0" friction="0"/>
     </joint>
-    <!-- JOINT: Connect base_link to ur5e mount (8 inches right of center) -->
+    <!-- JOINT: Connect turntable_disc_link to turntable_base_link -->
+    <joint name="${tf_prefix}disc_to_base" type="fixed">
+      <origin xyz="0 0 -0.1015" rpy="0 0 0"/>
+      <parent link="${tf_prefix}turntable_disc_link"/>
+      <child link="${tf_prefix}turntable_base_link"/>
+    </joint>
+    <!-- JOINT: Connect turntable_base_link to ur5e mount -->
     <joint name="${tf_prefix}base_to_mount" type="fixed">
-      <origin xyz="0.2032 0 0.057150" rpy="0 0 0"/>
-      <parent link="base_link"/>
+      <origin xyz="0.97035 0 0" rpy="0 0 0"/>
+      <parent link="${tf_prefix}turntable_base_link"/>
       <child link="${tf_prefix}ur5e_mount_link"/>
     </joint>
-    <!-- JOINT: Connect ur5e mount to ur5e base (on top of mount) -->
+    <!-- JOINT: Connect ur5e mount to ur5e base (on top of mount, adjusted for new mount frame) -->
     <joint name="${tf_prefix}mount_to_ur5e" type="fixed">
-      <origin xyz="0 0 0.057150" rpy="0 0 0"/>
+      <origin xyz="0 0 0.1143" rpy="0 0 0"/>
       <parent link="${tf_prefix}ur5e_mount_link"/>
       <child link="${tf_prefix}ur_base_link"/>
