Commit message: Working correct urdf for the cell - for RViz as well as physical hardware. URDFs need to be cleaned and well written again. Work in Progress.

File: inspection_cell_description/urdf/inspection_cell.urdf (robot description, URDF)
Before this commit: robot inspection_cell, 24 links, 24 joints
Links:
- removed link world
- link table_link: geometry collision box size=2.4384 1.524 0.903; visual mesh filename=package://inspection_cell_description/meshes/visual/table.d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
Joints:
- removed joint disc_to_base_inertia
- removed joint table_to_object
- removed joint world_joint
- removed joint world_to_table
- added joint object_to_disc: type fixed, parent object_frame, child turntable_disc_link, origin xyz=0 0 0 rpy=0 0 0
- added joint ur5e_mount_to_table: type fixed, parent ur5e_mount_link, child table_link, origin xyz=0 0 0 rpy=0 0 0
- joint turntable_disc_joint: child turntable_disc_link -> turntable_base_link_inertia; origin xyz=0 0 0 rpy=0 0 0 -> xyz=0 0 -0.1015 rpy=0 0 0; parent object_frame -> turntable_disc_link

File: inspection_cell_description/urdf/inspection_cell.urdf.xacro (robot description, xacro)
@@ -76,12 +76,7 @@
    <xacro:property name="hash" value="$(arg hash)" />
    <!-- ================================================================ -->
-   <!-- WORLD LINK -->
+   <!-- OBJECT FRAME -->
    <!-- ================================================================ -->
-   <link name="world"/>
-   <joint name="world_joint" type="fixed">
-      <origin xyz="0 0 0" rpy="0 0 0"/>
-      <parent link="world" />
-      <child link="table_link" />
-   </joint>
+   <link name="object_frame"/>
    <!-- ================================================================ -->
    <!-- GROUND PLANE FOR SIMULATION -->
@@ -107,5 +102,5 @@
      <joint name="ground_plane_joint" type="fixed">
        <origin xyz="0 0 -0.01" rpy="0 0 0"/>
-       <parent link="world"/>
+       <parent link="object_frame"/>
        <child link="ground_plane"/>
      </joint>
@@ -117,5 +112,5 @@
      name="$(arg name)"
      tf_prefix="$(arg tf_prefix)"
-     parent="world"
+     parent="object_frame"
      joint_limits_parameters_file="$(arg joint_limit_params)"
      kinematics_parameters_file="$(arg kinematics_params)"

File: inspection_cell_description/urdf/inspection_cell_macro.xacro (robot description, xacro)
@@ -128,12 +128,10 @@
       </visual>
       <collision>
-        <origin xyz="0 0 -0.4572" rpy="0 0 0"/>
-        <geometry>
-          <mesh filename="package://inspection_cell_description/meshes/collision/table.stl"/>
-        </geometry>
-      </collision>
-    </link>
-    <!-- Object Frame - ROOT of unified kinematic chain for object-centric planning -->
-    <link name="${tf_prefix}object_frame"/>
+        <origin xyz="0 0 -0.4515" rpy="0 0 0"/>
+        <geometry>
+          <box size="2.4384 1.524 0.903"/>
+        </geometry>
+      </collision>
+    </link>
     <!-- Turntable Disc Link - DOF 1 (Rotates the object) -->
     <link name="${tf_prefix}turntable_disc_link">
@@ -482,21 +480,20 @@
     <!-- JOINTS - OBJECT-CENTRIC UNIFIED KINEMATIC CHAIN -->
     <!-- ================================================================ -->
-    <!-- Table Link - Fixed to world for visualization -->
-    <joint name="${tf_prefix}world_to_table" type="fixed">
+    <!-- Object Frame - ROOT of unified kinematic chain
+    <joint name="${tf_prefix}world_to_object" type="fixed">
+      <origin xyz="-0.76835 0 0.1015" rpy="0 0 0"/>
+      <parent link="${parent}"/>
+      <child link="${tf_prefix}object_frame"/>
+    </joint> -->
+    <joint name="${tf_prefix}object_to_disc" type="fixed">
+      <parent link="${parent}"/>
+      <child link="${tf_prefix}turntable_disc_link"/>
       <origin xyz="0 0 0" rpy="0 0 0"/>
-      <parent link="${parent}"/>
-      <child link="${tf_prefix}table_link"/>
-    </joint>
-    <!-- Object Frame - ROOT of unified kinematic chain -->
-    <joint name="${tf_prefix}table_to_object" type="fixed">
-      <origin xyz="-0.76835 0 0.1015" rpy="0 0 0"/>  <!-- Position object above turntable -->
-      <parent link="${tf_prefix}table_link"/>
-      <child link="${tf_prefix}object_frame"/>
     </joint>
     <!-- DOF 1: Turntable Disc Rotation - Object rotates with disc -->
     <joint name="${tf_prefix}turntable_disc_joint" type="revolute">
-      <parent link="${tf_prefix}object_frame"/>
-      <child link="${tf_prefix}turntable_disc_link"/>
-      <origin xyz="0 0 0" rpy="0 0 0"/>  <!-- Disc below object -->
+      <parent link="${tf_prefix}turntable_disc_link"/>
+      <child link="${tf_prefix}turntable_base_link_inertia"/>
+      <origin xyz="0 0 -0.1015" rpy="0 0 0"/>   <!-- Position disc below object -->
       <axis xyz="0 0 1"/>
       <limit
@@ -515,9 +512,9 @@
     </joint>
     <!-- Turntable Base Link Inertia - Coordinate alignment -->
-    <joint name="${tf_prefix}disc_to_base_inertia" type="fixed">
-      <parent link="${tf_prefix}turntable_disc_link"/>
+    <!-- <joint name="${tf_prefix}disc_to_base_inertia" type="fixed">
+      <parent link="${tf_prefix}turntable_base_link"/>
       <child link="${tf_prefix}turntable_base_link_inertia"/>
-      <origin xyz="0 0 -0.1015" rpy="0 0 0"/>
-    </joint>
+      <origin xyz="-0.76835 0 0" rpy="0 0 0"/>
+    </joint> -->
     <!-- Turntable Base Link - Physical base structure -->
     <joint name="${tf_prefix}base_inertia_to_base" type="fixed">
@@ -526,4 +523,9 @@
       <origin xyz="0 0 0" rpy="0 0 0"/>
     </joint>
+    <joint name="${tf_prefix}ur5e_mount_to_table" type="fixed">
+      <origin xyz="0 0 0" rpy="0 0 0"/>
+      <parent link="${tf_prefix}ur5e_mount_link"/>
+      <child link="${tf_prefix}table_link"/>
+    </joint>
     <!-- UR5e Mount - Connected via turntable base -->
     <joint name="${tf_prefix}base_to_ur_mount" type="fixed">
@@ -536,5 +538,5 @@
       <parent link="${tf_prefix}ur5e_mount_link"/>
       <child link="${tf_prefix}ur_base_link"/>
-      <origin xyz="0 0 0.1143" rpy="0 0 0"/>
+      <origin xyz="0 0 0.1143" rpy="0 0 ${pi}"/>
     </joint>
     <!-- UR Coordinate System Alignment -->

Commit message: WIP - added the moveit_servo node but its still not working as it displays the ee frame as panda_link8 and ours is eoat_caera_link. Creating a new moveit config package to remove all the clutter.

File: inspection_cell_description/urdf/inspection_cell.urdf (robot description, URDF)
Before this commit: robot inspection_cell, 23 links, 22 joints
Joints:
- joint mount_to_ur: origin xyz=0 0 0.1143 rpy=0 0 0 -> xyz=0 0 0.1143 rpy=0 0 3.141592653589793

File: inspection_cell_description/urdf/inspection_cell_macro.xacro (robot description, xacro)
@@ -480,10 +480,5 @@
     <!-- JOINTS - OBJECT-CENTRIC UNIFIED KINEMATIC CHAIN -->
     <!-- ================================================================ -->
-    <!-- Object Frame - ROOT of unified kinematic chain
-    <joint name="${tf_prefix}world_to_object" type="fixed">
-      <origin xyz="-0.76835 0 0.1015" rpy="0 0 0"/>
-      <parent link="${parent}"/>
-      <child link="${tf_prefix}object_frame"/>
-    </joint> -->
+    <!-- Object Frame - ROOT of unified kinematic chain -->
     <joint name="${tf_prefix}object_to_disc" type="fixed">
       <parent link="${parent}"/>

File: inspection_cell_moveit_config/config/inspection_cell.ros2_control.xacro (robot description, xacro)
@@ -2,5 +2,5 @@
 <robot xmlns:xacro="http://www.ros.org/wiki/xacro">
     <xacro:macro name="inspection_cell_ros2_control" params="name initial_positions_file">
-        <xacro:property name="initial_positions" value="${xacro.load_yaml(initial_positions_file)['initial_positions']}"/>
+        <xacro:property name="initial_positions" value="${load_yaml(initial_positions_file)['initial_positions']}"/>
         <ros2_control name="${name}" type="system">
             <hardware>

Commit message: Corrected .urdf file.

File: inspection_cell_description/urdf/inspection_cell.urdf (robot description, URDF)
Before this commit: robot inspection_cell, 23 links, 22 joints
Joints:
- removed joint base_link-base_fixed_joint
- removed joint base_link-base_link_inertia
- added joint ur_base_link-base_fixed_joint: type fixed, parent ur_base_link, child base, origin xyz=0 0 0 rpy=0 0 3.141592653589793
- added joint ur_base_link-base_link_inertia: type fixed, parent ur_base_link, child base_link_inertia, origin xyz=0 0 0 rpy=0 0 3.141592653589793
- joint base_to_ur_mount: origin xyz=0.97035 0 0 rpy=0 0 0 -> xyz=0.9906 0 0 rpy=0 0 0
- joint ur5e_mount_to_table: origin xyz=0 0 0 rpy=0 0 0 -> xyz=-1.4732 -0.6096 0 rpy=0 0 0

Commit message: planning

File: inspection_cell_description/urdf/inspection_cell.urdf (robot description, URDF)
Before this commit: robot inspection_cell, 23 links, 22 joints
Joints:
- joint base_to_ur_mount: origin xyz=0.9906 0 0 rpy=0 0 0 -> xyz=0.75 0 0 rpy=0 0 0
- joint eoat_camera_joint: origin xyz=0 0 0.125 rpy=1.5707963267948966 3.141592653589793 -1.5707963267948966 -> xyz=0 0 0.125 rpy=1.5707963267948966 0 -1.5707963267948966

File: inspection_cell_description/urdf/inspection_cell_macro.xacro (robot description, xacro)
@@ -527,5 +527,5 @@
       <parent link="${tf_prefix}turntable_base_link"/>
       <child link="${tf_prefix}ur5e_mount_link"/>
-      <origin xyz="0.9906 0 0" rpy="0 0 0"/>
+      <origin xyz="0.75 0 0" rpy="0 0 0"/>
     </joint>
     <!-- UR5e Base - Mounted on mount block -->
