Commit message: Fixed almost everything w.r.t the URDF. Added 'inspection_cell_forward_position_controller' and configured the 'cell_servo.yaml' correctly.

File: inspection_cell_description/urdf/inspection_cell.urdf.xacro (robot description, xacro)
@@ -149,5 +149,5 @@
      hash="${hash}"
      >
-     <!-- Position robot in the world -->
+     <!-- Position robot -->
      <ur5e_origin xyz="0 0 0" rpy="0 0 0" />
      <turntable_origin xyz="0.75 0 0" rpy="0 0 0" />
@@ -157,5 +157,5 @@
    <!-- ================================================================ -->
    <xacro:if value="$(arg sim_gazebo)">
-    <gazebo reference="world">
+    <gazebo reference="object_frame">
     </gazebo>
     <gazebo>
@@ -169,5 +169,5 @@
    <!-- ================================================================ -->
    <xacro:if value="$(arg sim_ignition)">
-    <gazebo reference="world">
+    <gazebo reference="object_frame">
     </gazebo>
     <gazebo>

File: inspection_cell_description/urdf/inspection_cell_macro.xacro (robot description, xacro)
@@ -201,5 +201,5 @@
     <!-- UR5E ROBOT ARM LINKS (DOF 2-7) - Following Universal Robots Structure -->
     <!-- ================================================================ -->
-    <!-- UR base_link (mounted to ur5e_mount) -->
+    <!-- ur_base_link (mounted to ur5e_mount) -->
     <link name="${tf_prefix}ur_base_link"/>
     <!-- UR base_link_inertia (maintains UR internal coordinate system) -->
@@ -536,5 +536,5 @@
     </joint>
     <!-- UR Coordinate System Alignment -->
-    <joint name="${tf_prefix}base_link-base_link_inertia" type="fixed">
+    <joint name="${tf_prefix}ur_base_link-base_link_inertia" type="fixed">
       <parent link="${tf_prefix}ur_base_link"/>
       <child link="${tf_prefix}base_link_inertia"/>
@@ -650,5 +650,5 @@
       <origin xyz="0 0 0" rpy="${pi} 0 0"/>
     </joint>
-    <joint name="${tf_prefix}base_link-base_fixed_joint" type="fixed">
+    <joint name="${tf_prefix}ur_base_link-base_fixed_joint" type="fixed">
       <origin xyz="0 0 0" rpy="0 0 ${pi}"/>
       <parent link="${tf_prefix}ur_base_link"/>

Commit message: multiple cells

File: inspection_cell_description/urdf/inspection_cell.urdf.xacro (robot description, xacro)
@@ -6,7 +6,17 @@
    <xacro:arg name="name" default="inspection_cell"/>
    <!-- ================================================================ -->
+   <!-- CELL PARAMETER -->
+   <!-- ================================================================ -->
+   <xacro:arg name="cell" default="alpha"/>
+   <xacro:property name="cell" value="$(arg cell)"/>
+   <!-- ================================================================ -->
    <!-- IMPORT MAIN MACRO -->
    <!-- ================================================================ -->
-   <xacro:include filename="$(find inspection_cell_description)/urdf/inspection_cell_macro.xacro"/>
+   <xacro:if value="${cell == 'alpha'}">
+    <xacro:include filename="$(find inspection_cell_description)/urdf/inspection_cell_alpha.urdf.xacro"/>
+   </xacro:if>
+   <xacro:if value="${cell == 'beta'}">
+    <xacro:include filename="$(find inspection_cell_description)/urdf/inspection_cell_beta.urdf.xacro"/>
+   </xacro:if>
    <!-- ================================================================ -->
    <!-- SYSTEM TYPE PARAMETER -->
@@ -25,8 +35,8 @@
    <!-- CONFIGURATION FILES -->
    <!-- ================================================================ -->
-   <xacro:arg name="joint_limit_params" default="$(find inspection_cell_description)/config/joint_limits.yaml"/>
-   <xacro:arg name="kinematics_params" default="$(find inspection_cell_description)/config/default_kinematics.yaml"/>
-   <xacro:arg name="physical_params" default="$(find inspection_cell_description)/config/physical_parameters.yaml"/>
-   <xacro:arg name="visual_params" default="$(find inspection_cell_description)/config/visual_parameters.yaml"/>
+   <xacro:arg name="joint_limit_params" default="$(find inspection_cell_description)/config/cell_${cell}/joint_limits.yaml"/>
+   <xacro:arg name="kinematics_params" default="$(find inspection_cell_description)/config/cell_${cell}/kinematics.yaml"/>
+   <xacro:arg name="physical_params" default="$(find inspection_cell_description)/config/cell_${cell}/physical_parameters.yaml"/>
+   <xacro:arg name="visual_params" default="$(find inspection_cell_description)/config/cell_${cell}/visual_parameters.yaml"/>
    <xacro:arg name="transmission_hw_interface" default=""/>
    <!-- ================================================================ -->
@@ -34,5 +44,10 @@
    <!-- ================================================================ -->
    <xacro:arg name="headless_mode" default="false" />
-   <xacro:arg name="robot_ip" default="0.0.0.0" />
+   <xacro:if value="${cell == 'alpha'}">
+    <xacro:arg name="robot_ip" default="192.168.1.102" />
+   </xacro:if>
+   <xacro:if value="${cell == 'beta'}">
+    <xacro:arg name="robot_ip" default="192.168.1.103" />
+   </xacro:if>
    <xacro:arg name="script_filename" default=""/>
    <xacro:arg name="output_recipe_filename" default=""/>
@@ -69,5 +84,5 @@
    <!-- INITIAL POSITION FOR SIMULATIONS -->
    <!-- ================================================================ -->
-   <xacro:arg name="initial_positions_file" default="$(find inspection_cell_description)/config/initial_positions.yaml"/>
+   <xacro:arg name="initial_positions_file" default="$(find inspection_cell_description)/config/cell_${cell}/initial_positions.yaml"/>
    <!-- Convert to property to use substitution in function -->
    <xacro:property name="initial_positions_file" default="$(arg initial_positions_file)"/>

Commit message: having difficulties with move_group.launch.py

File: inspection_cell_description/urdf/inspection_cell.urdf.xacro (robot description, xacro)
@@ -35,8 +35,8 @@
    <!-- CONFIGURATION FILES -->
    <!-- ================================================================ -->
-   <xacro:arg name="joint_limit_params" default="$(find inspection_cell_description)/config/cell_${cell}/joint_limits.yaml"/>
-   <xacro:arg name="kinematics_params" default="$(find inspection_cell_description)/config/cell_${cell}/kinematics.yaml"/>
-   <xacro:arg name="physical_params" default="$(find inspection_cell_description)/config/cell_${cell}/physical_parameters.yaml"/>
-   <xacro:arg name="visual_params" default="$(find inspection_cell_description)/config/cell_${cell}/visual_parameters.yaml"/>
+   <xacro:arg name="joint_limit_params" default="$(find inspection_cell_description)/config/${cell}/joint_limits.yaml"/>
+   <xacro:arg name="kinematics_params" default="$(find inspection_cell_description)/config/${cell}/kinematics.yaml"/>
+   <xacro:arg name="physical_params" default="$(find inspection_cell_description)/config/${cell}/physical_parameters.yaml"/>
+   <xacro:arg name="visual_params" default="$(find inspection_cell_description)/config/${cell}/visual_parameters.yaml"/>
    <xacro:arg name="transmission_hw_interface" default=""/>
    <!-- ================================================================ -->
@@ -44,10 +44,5 @@
    <!-- ================================================================ -->
    <xacro:arg name="headless_mode" default="false" />
-   <xacro:if value="${cell == 'alpha'}">
-    <xacro:arg name="robot_ip" default="192.168.1.102" />
-   </xacro:if>
-   <xacro:if value="${cell == 'beta'}">
-    <xacro:arg name="robot_ip" default="192.168.1.103" />
-   </xacro:if>
+   <xacro:arg name="robot_ip" default="192.168.0.102" />
    <xacro:arg name="script_filename" default=""/>
    <xacro:arg name="output_recipe_filename" default=""/>
@@ -84,5 +79,5 @@
    <!-- INITIAL POSITION FOR SIMULATIONS -->
    <!-- ================================================================ -->
-   <xacro:arg name="initial_positions_file" default="$(find inspection_cell_description)/config/cell_${cell}/initial_positions.yaml"/>
+   <xacro:arg name="initial_positions_file" default="$(find inspection_cell_description)/config/${cell}/initial_positions.yaml"/>
    <!-- Convert to property to use substitution in function -->
    <xacro:property name="initial_positions_file" default="$(arg initial_positions_file)"/>

File: inspection_cell_description/urdf/inspection_cell_alpha.urdf.xacro (robot description, xacro)
@@ -47,5 +47,5 @@
     sim_ignition:=false
     headless_mode:=false
-    initial_positions:=${dict(turntable_disc_joint=0.0,shoulder_pan_joint=0.0,shoulder_lift_joint=-1.57,elbow_joint=1.57,wrist_1_joint=-1.57,wrist_2_joint=-1.57,wrist_3_joint=0.0)}
+    initial_positions:=${dict(turntable_disc_joint=0.0,shoulder_pan_joint=0.0,shoulder_lift_joint=0.0,elbow_joint=0.0,wrist_1_joint=0.0,wrist_2_joint=0.0,wrist_3_joint=0.0)}
     use_tool_communication:=false
     tool_voltage:=0
@@ -91,5 +91,5 @@
         tf_prefix="${tf_prefix}"
         hash="${hash}"
-        robot_ip="${robot_ip}"
+        robot_ip="192.168.0.12"
         script_filename="${script_filename}"
         output_recipe_filename="${output_recipe_filename}"

File: inspection_cell_moveit_config/config/inspection_cell.ros2_control.xacro (robot description, xacro)
@@ -2,5 +2,5 @@
 <robot xmlns:xacro="http://www.ros.org/wiki/xacro">
     <xacro:macro name="inspection_cell_ros2_control" params="name initial_positions_file">
-        <xacro:property name="initial_positions" value="${xacro.load_yaml(initial_positions_file)['initial_positions']}"/>
+        <xacro:property name="initial_positions" value="${xacro.load_yaml(initial_positions_file)}"/>
         <ros2_control name="${name}" type="system">
             <hardware>
