Commit message: added planning volume

File: inspection_cell_description/urdf/inspection_cell_alpha.urdf.xacro (robot description, xacro)
@@ -478,4 +478,54 @@
     <link name="${tf_prefix}turntable_base"/>
     <!-- ================================================================ -->
+    <!-- PLANNING VOLUME -->
+    <!-- ================================================================ -->
+    <!-- Define your planning volume dimensions -->
+    <xacro:property name="planning_width" value="0.620"/>   <!-- X dimension -->
+    <xacro:property name="planning_depth" value="0.620"/>   <!-- Y dimension -->
+    <xacro:property name="planning_height" value="1.000"/>  <!-- Z dimension -->
+    <xacro:property name="wall_thickness" value="0.001"/>
+    <link name="${tf_prefix}planning_volume">
+      <!-- Front wall (positive X) -->
+      <collision name="wall_front">
+      <origin xyz="${planning_width/2} 0 ${planning_height/2}" rpy="0 0 0"/>
+      <geometry>
+        <box size="${wall_thickness} ${planning_depth} ${planning_height}"/>
+      </geometry>
+      </collision>
+      <!-- Back wall (negative X) -->
+      <collision name="wall_back">
+      <origin xyz="${-planning_width/2} 0 ${planning_height/2}" rpy="0 0 0"/>
+      <geometry>
+        <box size="${wall_thickness} ${planning_depth} ${planning_height}"/>
+      </geometry>
+      </collision>
+      <!-- Left wall (positive Y) -->
+      <collision name="wall_left">
+      <origin xyz="0 ${planning_depth/2} ${planning_height/2}" rpy="0 0 0"/>
+      <geometry>
+        <box size="${planning_width} ${wall_thickness} ${planning_height}"/>
+      </geometry>
+      </collision>
+      <!-- Right wall (negative Y) -->
+      <collision name="wall_right">
+      <origin xyz="0 ${-planning_depth/2} ${planning_height/2}" rpy="0 0 0"/>
+      <geometry>
+        <box size="${planning_width} ${wall_thickness} ${planning_height}"/>
+      </geometry>
+      </collision>
+      <!-- Ceiling (positive Z) -->
+      <collision name="wall_ceiling">
+        <origin xyz="0 0 ${planning_height}" rpy="0 0 0"/>
+        <geometry>
+          <box size="${planning_width} ${planning_depth} ${wall_thickness}"/>
+        </geometry>
+      </collision>
+    </link>
+    <joint name="${tf_prefix}turntable_base_to_planning_volume" type="fixed">
+      <parent link="${tf_prefix}turntable_base_link"/>
+      <child link="${tf_prefix}planning_volume"/>
+      <origin xyz="0.325 0 0" rpy="0 0 0"/>
+    </joint>
+    <!-- ================================================================ -->
     <!-- JOINTS - OBJECT-CENTRIC UNIFIED KINEMATIC CHAIN -->
     <!-- ================================================================ -->

Commit message: added camera_depth_optical_frame

File: inspection_cell_description/urdf/inspection_cell_alpha.urdf.xacro (robot description, xacro)
@@ -469,4 +469,19 @@
       </inertial>
     </link>
+    <link name="${tf_prefix}camera_depth_optical_frame">
+      <visual>
+        <origin xyz="0 0 0" rpy="0 ${radians(-90)} 0"/>
+        <geometry>
+          <cylinder radius="0.015" length="0.030"/>
+        </geometry>
+        <material name="depth_camera_optical_frame_material"/>
+      </visual>
+      <collision>
+        <origin xyz="0 0 0" rpy="0 ${radians(-90)} 0"/>
+        <geometry>
+          <cylinder radius="0.015" length="0.030"/>
+        </geometry>
+      </collision>
+    </link>
     <!-- ================================================================ -->
     <!-- INDUSTRIAL COMPATIBILITY FRAMES -->
@@ -738,4 +753,9 @@
       <origin xyz="0 0 0.125" rpy="${radians(90)} ${radians(0)} ${radians(-90)}"/>
     </joint>
+    <joint name="${tf_prefix}camera_depth_optical_joint" type="fixed">
+      <parent link="${tf_prefix}eoat_base_link"/>
+      <child link="${tf_prefix}camera_depth_optical_frame"/>
+      <origin xyz="-0.080 0 0.06" rpy="0 ${radians(-180)} 0"/>
+    </joint>
     <!-- ================================================================ -->
     <!-- INDUSTRIAL COMPATIBILITY FRAMES -->

Commit message: added load_yaml and updated depth camera frame  joint

File: inspection_cell_description/urdf/inspection_cell_alpha.urdf.xacro (robot description, xacro)
@@ -756,5 +756,5 @@
       <parent link="${tf_prefix}eoat_base_link"/>
       <child link="${tf_prefix}camera_depth_optical_frame"/>
-      <origin xyz="-0.080 0 0.06" rpy="0 ${radians(-180)} 0"/>
+      <origin xyz="-0.080 0 0.06" rpy="${radians(90)} 0 ${radians(-90)}"/>
     </joint>
     <!-- ================================================================ -->

Commit message: fixed tf tree for alpha and beta

File: inspection_cell_description/urdf/inspection_cell_alpha.urdf.xacro (robot description, xacro)
@@ -469,7 +469,7 @@
       </inertial>
     </link>
-    <link name="${tf_prefix}camera_depth_optical_frame">
-      <visual>
-        <origin xyz="0 0 0" rpy="0 ${radians(-90)} 0"/>
+    <link name="${tf_prefix}camera_link">
+      <visual>
+        <origin xyz="0 0 0" rpy="0 ${radians(90)} 0"/>
         <geometry>
           <cylinder radius="0.015" length="0.030"/>
@@ -478,5 +478,5 @@
       </visual>
       <collision>
-        <origin xyz="0 0 0" rpy="0 ${radians(-90)} 0"/>
+        <origin xyz="0 0 0" rpy="0 ${radians(90)} 0"/>
         <geometry>
           <cylinder radius="0.015" length="0.030"/>
@@ -755,6 +755,6 @@
     <joint name="${tf_prefix}camera_depth_optical_joint" type="fixed">
       <parent link="${tf_prefix}eoat_base_link"/>
-      <child link="${tf_prefix}camera_depth_optical_frame"/>
-      <origin xyz="-0.080 0 0.06" rpy="${radians(90)} 0 ${radians(-90)}"/>
+      <child link="${tf_prefix}camera_link"/>
+      <origin xyz="-0.080 0 0.06" rpy="0 ${radians(180)} 0"/>
     </joint>
     <!-- ================================================================ -->

File: inspection_cell_description/urdf/inspection_cell_beta.urdf.xacro (robot description, xacro)
@@ -469,4 +469,19 @@
       </inertial>
     </link>
+    <link name="${tf_prefix}camera_link">
+      <visual>
+        <origin xyz="0 0 0" rpy="0 ${radians(90)} 0"/>
+        <geometry>
+          <cylinder radius="0.015" length="0.030"/>
+        </geometry>
+        <material name="depth_camera_optical_frame_material"/>
+      </visual>
+      <collision>
+        <origin xyz="0 0 0" rpy="0 ${radians(90)} 0"/>
+        <geometry>
+          <cylinder radius="0.015" length="0.030"/>
+        </geometry>
+      </collision>
+    </link>
     <!-- ================================================================ -->
     <!-- INDUSTRIAL COMPATIBILITY FRAMES -->
@@ -738,4 +753,9 @@
       <origin xyz="0 0 0.125" rpy="${radians(90)} ${radians(0)} ${radians(-90)}"/>
     </joint>
+    <joint name="${tf_prefix}camera_depth_optical_joint" type="fixed">
+      <parent link="${tf_prefix}eoat_base_link"/>
+      <child link="${tf_prefix}camera_link"/>
+      <origin xyz="-0.080 0 0.06" rpy="0 ${radians(180)} 0"/>
+    </joint>
     <!-- ================================================================ -->
     <!-- INDUSTRIAL COMPATIBILITY FRAMES -->

Commit message: changed orientation of axis of depthcamera for alpha cell

File: inspection_cell_description/urdf/inspection_cell_alpha.urdf.xacro (robot description, xacro)
@@ -756,5 +756,5 @@
       <parent link="${tf_prefix}eoat_base_link"/>
       <child link="${tf_prefix}camera_link"/>
-      <origin xyz="-0.080 0 0.06" rpy="0 ${radians(180)} 0"/>
+      <origin xyz="0 0 0.06" rpy="0 0 ${radians(180)}"/>
     </joint>
     <!-- ================================================================ -->

File: inspection_cell_description/urdf/inspection_cell_beta.urdf.xacro (robot description, xacro)
@@ -27,5 +27,5 @@
   </material>
   <material name="vention_blue">
-    <color rgba="0.0 0.2 0.8 1.0"/>
+    <color rgba="0.122 0.184 0.09 1.0"/>
   </material>
   <xacro:macro name="inspection_cell" params="

Commit message: rotated the eaot_base_link pitch 180 degrees

File: inspection_cell_description/urdf/inspection_cell_alpha.urdf.xacro (robot description, xacro)
@@ -756,5 +756,5 @@
       <parent link="${tf_prefix}eoat_base_link"/>
       <child link="${tf_prefix}camera_link"/>
-      <origin xyz="0 0 0.06" rpy="0 0 ${radians(180)}"/>
+      <origin xyz="0 0 0.06" rpy="0 ${radians(180)} ${radians(180)}"/>
     </joint>
     <!-- ================================================================ -->

File: inspection_cell_description/urdf/inspection_cell_beta.urdf.xacro (robot description, xacro)
@@ -759,5 +759,5 @@
       <parent link="${tf_prefix}eoat_base_link"/>
       <child link="${tf_prefix}camera_link"/>
-      <origin xyz="-0.080 0 0.06" rpy="0 0 ${radians(180)}"/>
+      <origin xyz="-0.080 0 0.06" rpy="0 ${radians(180)} ${radians(180)}"/>
     </joint>
     <!-- ================================================================ -->

Commit message: instead of pitch it had to be roll of 180 degrees to reorient depth optical frame

File: inspection_cell_description/urdf/inspection_cell_alpha.urdf.xacro (robot description, xacro)
@@ -756,5 +756,5 @@
       <parent link="${tf_prefix}eoat_base_link"/>
       <child link="${tf_prefix}camera_link"/>
-      <origin xyz="0 0 0.06" rpy="0 ${radians(180)} ${radians(180)}"/>
+      <origin xyz="0 0 0.06" rpy="${radians(180)} 0 ${radians(180)}"/>
     </joint>
     <!-- ================================================================ -->

File: inspection_cell_description/urdf/inspection_cell_beta.urdf.xacro (robot description, xacro)
@@ -759,5 +759,5 @@
       <parent link="${tf_prefix}eoat_base_link"/>
       <child link="${tf_prefix}camera_link"/>
-      <origin xyz="-0.080 0 0.06" rpy="0 ${radians(180)} ${radians(180)}"/>
+      <origin xyz="-0.080 0 0.06" rpy="${radians(180)} 0 ${radians(180)}"/>
     </joint>
     <!-- ================================================================ -->

Commit message: fixed camera frame joint. need to improve visuals.

File: inspection_cell_description/urdf/inspection_cell_alpha.urdf.xacro (robot description, xacro)
@@ -413,5 +413,5 @@
         <origin xyz="0 0 0.024535"/>
         <geometry>
-          <cylinder radius="0.035" length="0.04907"/>
+          <cylinder radius="0.035" length="0.001"/>
         </geometry>
         <material name="eoat_black"/>
@@ -433,5 +433,5 @@
         <origin xyz="0 0 0.080"/>
         <geometry>
-          <cylinder radius="0.0325" length="0.160"/>
+          <cylinder radius="0.04" length="0.160"/>
         </geometry>
         <material name="eoat_black"/>
@@ -440,5 +440,5 @@
         <origin xyz="0 0 0.080"/>
         <geometry>
-          <cylinder radius="0.0325" length="0.160"/>
+          <cylinder radius="0.04" length="0.160"/>
         </geometry>
       </collision>
@@ -451,14 +451,14 @@
     <link name="${tf_prefix}eoat_body_link">
       <visual>
+        <origin xyz="0 0 0.035"/>
+        <geometry>
+          <box size="0.1, 0.1 0.1"/>
+        </geometry>
+        <material name="eoat_black"/>
+      </visual>
+      <collision>
         <origin xyz="0 0 0.0625"/>
         <geometry>
-          <box size="0.125 0.125 0.125"/>
-        </geometry>
-        <material name="eoat_black"/>
-      </visual>
-      <collision>
-        <origin xyz="0 0 0.0625"/>
-        <geometry>
-          <box size="0.125 0.125 0.125"/>
+          <box size="0.07, 0.07 0.07"/>
         </geometry>
       </collision>
@@ -741,15 +741,15 @@
       <parent link="${tf_prefix}eoat_base_link"/>
       <child link="${tf_prefix}eoat_top_link"/>
-      <origin xyz="0 0 0.04907" rpy="0 0 0"/>
+      <origin xyz="0 0 0.0" rpy="0 0 0"/>
     </joint>
     <joint name="${tf_prefix}eoat_body_joint" type="fixed">
       <parent link="${tf_prefix}eoat_base_link"/>
       <child link="${tf_prefix}eoat_body_link"/>
-      <origin xyz="0.050 0 0.125" rpy="${radians(90)} ${radians(180)} ${radians(-90)}"/>
+      <origin xyz="0.050 0 0.0475" rpy="${radians(90)} ${radians(180)} ${radians(-90)}"/>
     </joint>
     <joint name="${tf_prefix}eoat_camera_joint" type="fixed">
       <parent link="${tf_prefix}eoat_base_link"/>
       <child link="${tf_prefix}eoat_camera_link"/>
-      <origin xyz="0 0 0.125" rpy="${radians(90)} ${radians(0)} ${radians(-90)}"/>
+      <origin xyz="0.024475 0 0.0475" rpy="${radians(90)} ${radians(0)} ${radians(-90)}"/>
     </joint>
     <joint name="${tf_prefix}camera_depth_optical_joint" type="fixed">

Commit message: turntable position updated

File: inspection_cell_description/urdf/inspection_cell_alpha.urdf.xacro (robot description, xacro)
@@ -592,5 +592,5 @@
       <parent link="${tf_prefix}turntable_base_link"/>
       <child link="${tf_prefix}ur5e_mount_link"/>
-      <origin xyz="0.75 0 0" rpy="0 0 0"/>
+      <origin xyz="0.7493 0 0" rpy="0 0 0"/>
     </joint>
     <!-- UR5e Base - Mounted on mount block -->

Commit message: removing planning volume

File: inspection_cell_description/urdf/inspection_cell_alpha.urdf.xacro (robot description, xacro)
@@ -540,5 +540,5 @@
       <parent link="${tf_prefix}turntable_base_link"/>
       <child link="${tf_prefix}planning_volume"/>
-      <origin xyz="0.325 0 0" rpy="0 0 0"/>
+      <origin xyz="0 0 0" rpy="0 0 0"/>
     </joint>
     <!-- ================================================================ -->

Commit message: Corrected the URDF for alpha & beta - removed the undefined material  'depth_camera'. Fixed error in dimensions of the 'eoat camera'.

File: inspection_cell_description/urdf/inspection_cell_alpha.urdf.xacro (robot description, xacro)
@@ -453,5 +453,5 @@
         <origin xyz="0 0 0.035"/>
         <geometry>
-          <box size="0.1, 0.1 0.1"/>
+          <box size="0.1 0.1 0.1"/>
         </geometry>
         <material name="eoat_black"/>
@@ -460,5 +460,5 @@
         <origin xyz="0 0 0.0625"/>
         <geometry>
-          <box size="0.07, 0.07 0.07"/>
+          <box size="0.07 0.07 0.07"/>
         </geometry>
       </collision>
@@ -475,5 +475,4 @@
           <cylinder radius="0.015" length="0.030"/>
         </geometry>
-        <material name="depth_camera_optical_frame_material"/>
       </visual>
       <collision>

File: inspection_cell_description/urdf/inspection_cell_beta.urdf.xacro (robot description, xacro)
@@ -478,5 +478,4 @@
           <cylinder radius="0.015" length="0.030"/>
         </geometry>
-        <material name="depth_camera_optical_frame_material"/>
       </visual>
       <collision>

Commit message: removed planning volume

File: inspection_cell_description/urdf/inspection_cell_alpha.urdf.xacro (robot description, xacro)
@@ -499,41 +499,5 @@
     <xacro:property name="planning_height" value="1.000"/>  <!-- Z dimension -->
     <xacro:property name="wall_thickness" value="0.001"/>
-    <link name="${tf_prefix}planning_volume">
-      <!-- Front wall (positive X) -->
-      <collision name="wall_front">
-      <origin xyz="${planning_width/2} 0 ${planning_height/2}" rpy="0 0 0"/>
-      <geometry>
-        <box size="${wall_thickness} ${planning_depth} ${planning_height}"/>
-      </geometry>
-      </collision>
-      <!-- Back wall (negative X) -->
-      <collision name="wall_back">
-      <origin xyz="${-planning_width/2} 0 ${planning_height/2}" rpy="0 0 0"/>
-      <geometry>
-        <box size="${wall_thickness} ${planning_depth} ${planning_height}"/>
-      </geometry>
-      </collision>
-      <!-- Left wall (positive Y) -->
-      <collision name="wall_left">
-      <origin xyz="0 ${planning_depth/2} ${planning_height/2}" rpy="0 0 0"/>
-      <geometry>
-        <box size="${planning_width} ${wall_thickness} ${planning_height}"/>
-      </geometry>
-      </collision>
-      <!-- Right wall (negative Y) -->
-      <collision name="wall_right">
-      <origin xyz="0 ${-planning_depth/2} ${planning_height/2}" rpy="0 0 0"/>
-      <geometry>
-        <box size="${planning_width} ${wall_thickness} ${planning_height}"/>
-      </geometry>
-      </collision>
-      <!-- Ceiling (positive Z) -->
-      <collision name="wall_ceiling">
-        <origin xyz="0 0 ${planning_height}" rpy="0 0 0"/>
-        <geometry>
-          <box size="${planning_width} ${planning_depth} ${wall_thickness}"/>
-        </geometry>
-      </collision>
-    </link>
+    <link name="${tf_prefix}planning_volume"/>
     <joint name="${tf_prefix}turntable_base_to_planning_volume" type="fixed">
       <parent link="${tf_prefix}turntable_base_link"/>
