Commit message: altered cell beta to fit new setup

File: inspection_cell_description/urdf/inspection_cell_gamma.urdf.xacro (robot description, xacro)
@@ -25,4 +25,7 @@
   <material name="mount_black">
     <color rgba="0.1 0.1 0.1 1.0"/>
+  </material>
+  <material name="vention_blue">
+    <color rgba="0.122 0.184 0.09 1.0"/>
   </material>
   <xacro:macro name="inspection_cell" params="
@@ -122,13 +125,13 @@
     <link name="${tf_prefix}table_link">
       <visual>
-        <origin xyz="0 0 0" rpy="0 0 0"/>
-        <geometry>
-          <mesh filename="package://inspection_cell_description/meshes/visual/table.dae"/>
-        </geometry>
-      </visual>
-      <collision>
-        <origin xyz="1.2192 0.762 -0.4515" rpy="0 0 0"/>
-        <geometry>
-          <box size="2.4384 1.524 0.903"/>
+        <origin xyz="0 0 -0.0225" rpy="0 0 0"/>
+        <geometry>
+          <box size="1 2 0.045"/>
+        </geometry>
+      </visual>
+      <collision>
+        <origin xyz="0 0 -0.0225" rpy="0 0 0"/>
+        <geometry>
+          <box size="1 2 0.045"/>
         </geometry>
       </collision>
@@ -185,14 +188,14 @@
     <link name="${tf_prefix}ur5e_mount_link">
       <visual>
-        <origin xyz="0 0 0.05715" rpy="0 0 0"/>
-        <geometry>
-          <box size="0.1778 0.1778 0.1143"/>
+        <origin xyz="0 0 0.01125" rpy="0 0 0"/>
+        <geometry>
+          <box size="0.180 0.180 0.0225"/>
         </geometry>
         <material name="mount_black"/>
       </visual>
       <collision>
-        <origin xyz="0 0 0.05715" rpy="0 0 0"/>
-        <geometry>
-          <box size="0.1778 0.1778 0.1143"/>
+        <origin xyz="0 0 0.01125" rpy="0 0 0"/>
+        <geometry>
+          <box size="0.180 0.180 0.0225"/>
         </geometry>
       </collision>
@@ -413,5 +416,5 @@
         <origin xyz="0 0 0.024535"/>
         <geometry>
-          <cylinder radius="0.035" length="0.001"/>
+          <cylinder radius="0.035" length="0.04907"/>
         </geometry>
         <material name="eoat_black"/>
@@ -433,5 +436,5 @@
         <origin xyz="0 0 0.080"/>
         <geometry>
-          <cylinder radius="0.04" length="0.160"/>
+          <cylinder radius="0.0325" length="0.160"/>
         </geometry>
         <material name="eoat_black"/>
@@ -440,5 +443,5 @@
         <origin xyz="0 0 0.080"/>
         <geometry>
-          <cylinder radius="0.04" length="0.160"/>
+          <cylinder radius="0.0325" length="0.160"/>
         </geometry>
       </collision>
@@ -451,7 +454,7 @@
     <link name="${tf_prefix}eoat_body_link">
       <visual>
-        <origin xyz="0 0 0.035"/>
-        <geometry>
-          <box size="0.1, 0.1 0.1"/>
+        <origin xyz="0 0 0.0625"/>
+        <geometry>
+          <box size="0.125 0.125 0.125"/>
         </geometry>
         <material name="eoat_black"/>
@@ -460,5 +463,5 @@
         <origin xyz="0 0 0.0625"/>
         <geometry>
-          <box size="0.07, 0.07 0.07"/>
+          <box size="0.125 0.125 0.125"/>
         </geometry>
       </collision>
@@ -475,11 +478,12 @@
           <cylinder radius="0.015" length="0.030"/>
         </geometry>
-      </visual>
-      <!-- <collision>
+        <material name="depth_camera_optical_frame_material"/>
+      </visual>
+      <collision>
         <origin xyz="0 0 0" rpy="0 ${radians(90)} 0"/>
         <geometry>
           <cylinder radius="0.015" length="0.030"/>
         </geometry>
-      </collision> -->
+      </collision>
     </link>
     <!-- ================================================================ -->
@@ -495,14 +499,8 @@
     <!-- ================================================================ -->
     <!-- Define your planning volume dimensions -->
-    <xacro:property name="planning_width" value="0.620"/>   <!-- X dimension -->
-    <xacro:property name="planning_depth" value="0.620"/>   <!-- Y dimension -->
+    <xacro:property name="planning_width" value="1.000"/>   <!-- X dimension -->
+    <xacro:property name="planning_depth" value="1.000"/>   <!-- Y dimension -->
     <xacro:property name="planning_height" value="1.000"/>  <!-- Z dimension -->
     <xacro:property name="wall_thickness" value="0.001"/>
-    <link name="${tf_prefix}planning_volume"/>
-    <joint name="${tf_prefix}turntable_base_to_planning_volume" type="fixed">
-      <parent link="${tf_prefix}turntable_base_link"/>
-      <child link="${tf_prefix}planning_volume"/>
-      <origin xyz="0 0 0" rpy="0 0 0"/>
-    </joint>
     <!-- ================================================================ -->
     <!-- JOINTS - OBJECT-CENTRIC UNIFIED KINEMATIC CHAIN -->
@@ -544,8 +542,8 @@
       <parent link="${tf_prefix}turntable_base_link_inertia"/>
       <child link="${tf_prefix}turntable_base_link"/>
+      <origin xyz="0 0 0" rpy="0 0 ${-pi/2}"/>
+    </joint>
+    <joint name="${tf_prefix}ur5e_mount_to_table" type="fixed">
       <origin xyz="0 0 0" rpy="0 0 0"/>
-    </joint>
-    <joint name="${tf_prefix}ur5e_mount_to_table" type="fixed">
-      <origin xyz="-1.4732 -0.6096 0" rpy="0 0 0"/>
       <parent link="${tf_prefix}ur5e_mount_link"/>
       <child link="${tf_prefix}table_link"/>
@@ -555,5 +553,5 @@
       <parent link="${tf_prefix}turntable_base_link"/>
       <child link="${tf_prefix}ur5e_mount_link"/>
-      <origin xyz="0.762 0 0" rpy="0 0 0"/>
+      <origin xyz="0 0.7287 0" rpy="0 0 0"/>
     </joint>
     <!-- UR5e Base - Mounted on mount block -->
@@ -561,5 +559,5 @@
       <parent link="${tf_prefix}ur5e_mount_link"/>
       <child link="${tf_prefix}ur_base_link"/>
-      <origin xyz="0 0 0.0693" rpy="0 0 ${pi/2}"/>
+      <origin xyz="0 0 0.0225" rpy="0 0 ${pi}"/>
     </joint>
     <!-- UR Coordinate System Alignment -->
@@ -704,20 +702,20 @@
       <parent link="${tf_prefix}eoat_base_link"/>
       <child link="${tf_prefix}eoat_top_link"/>
-      <origin xyz="0 0 0.0" rpy="0 0 0"/>
+      <origin xyz="0 0 0.04907" rpy="0 0 0"/>
     </joint>
     <joint name="${tf_prefix}eoat_body_joint" type="fixed">
       <parent link="${tf_prefix}eoat_base_link"/>
       <child link="${tf_prefix}eoat_body_link"/>
-      <origin xyz="0.050 0 0.0475" rpy="${radians(90)} ${radians(180)} ${radians(-90)}"/>
+      <origin xyz="0.050 0 0.125" rpy="${radians(90)} ${radians(180)} ${radians(-90)}"/>
     </joint>
     <joint name="${tf_prefix}eoat_camera_joint" type="fixed">
       <parent link="${tf_prefix}eoat_base_link"/>
       <child link="${tf_prefix}eoat_camera_link"/>
-      <origin xyz="0.024475 0 0.0475" rpy="${radians(90)} ${radians(0)} ${radians(-90)}"/>
+      <origin xyz="0 0 0.125" rpy="${radians(90)} ${radians(0)} ${radians(-90)}"/>
     </joint>
     <joint name="${tf_prefix}camera_depth_optical_joint" type="fixed">
       <parent link="${tf_prefix}eoat_base_link"/>
       <child link="${tf_prefix}camera_link"/>
-      <origin xyz="-0.050287 0 -0.01232" rpy="${radians(180)} 0 ${radians(180)}"/>
+      <origin xyz="-0.023 0 0.033" rpy="${radians(180)} 0 ${radians(180)}"/>
     </joint>
     <!-- ================================================================ -->
