Commit message: jazzy migration

File: inspection_cell_description/urdf/inspection_cell.ros2_control.xacro (robot description, xacro)
@@ -22,4 +22,5 @@
     non_blocking_read:=true
     keep_alive_count:=2
+    robot_receive_timeout:=0.04
     hash
     ">
@@ -72,4 +73,5 @@
           <param name="tool_tcp_port">${tool_tcp_port}</param>
           <param name="keep_alive_count">${keep_alive_count}</param>
+          <param name="robot_receive_timeout">${robot_receive_timeout}</param>
         </xacro:unless>
       </hardware>

File: inspection_cell_description/urdf/inspection_cell.urdf.xacro (robot description, xacro)
@@ -54,4 +54,5 @@
    <xacro:arg name="non_blocking_read" default="true"/>
    <xacro:arg name="keep_alive_count" default="2"/>
+   <xacro:arg name="robot_receive_timeout" default="0.04"/>
    <xacro:arg name="hash" default="calib_unified_7dof_12345678901234567890"/>
    <!-- ================================================================ -->
@@ -155,4 +156,5 @@
      non_blocking_read="$(arg non_blocking_read)"
      keep_alive_count="$(arg keep_alive_count)"
+     robot_receive_timeout="$(arg robot_receive_timeout)"
      hash="${hash}"
      >

File: inspection_cell_description/urdf/inspection_cell_alpha.urdf.xacro (robot description, xacro)
@@ -68,4 +68,5 @@
     non_blocking_read:=true
     keep_alive_count:=2
+    robot_receive_timeout:=0.04
     hash:=calib_unified_7dof_12345678901234567890
     ">
@@ -102,4 +103,5 @@
         non_blocking_read="${non_blocking_read}"
         keep_alive_count="${keep_alive_count}"
+        robot_receive_timeout="${robot_receive_timeout}"
         use_tool_communication="${use_tool_communication}"
         tool_voltage="${tool_voltage}"

File: inspection_cell_description/urdf/inspection_cell_beta.urdf.xacro (robot description, xacro)
@@ -68,4 +68,5 @@
     non_blocking_read:=true
     keep_alive_count:=2
+    robot_receive_timeout:=0.04
     hash:=calib_unified_7dof_12345678901234567890
     ">
@@ -102,4 +103,5 @@
         non_blocking_read="${non_blocking_read}"
         keep_alive_count="${keep_alive_count}"
+        robot_receive_timeout="${robot_receive_timeout}"
         use_tool_communication="${use_tool_communication}"
         tool_voltage="${tool_voltage}"
@@ -660,5 +662,5 @@
       <parent link="${tf_prefix}eoat_camera_link"/>
       <child link="${tf_prefix}camera_link"/>
-      <origin xyz="-0.0805 0.009 0.0984" rpy="${radians(90)} ${radians(-63.435)} ${radians(0)}"/>
+      <origin xyz="-0.0805 0.009 0.0984" rpy="${radians(0)} ${radians(-63.435)} ${radians(0)}"/>
     </joint>
     <!-- ================================================================ -->

File: inspection_cell_description/urdf/inspection_cell_gamma.urdf.xacro (robot description, xacro)
@@ -71,4 +71,5 @@
     non_blocking_read:=true
     keep_alive_count:=2
+    robot_receive_timeout:=0.04
     hash:=calib_unified_7dof_12345678901234567890
     ">
@@ -105,4 +106,5 @@
         non_blocking_read="${non_blocking_read}"
         keep_alive_count="${keep_alive_count}"
+        robot_receive_timeout="${robot_receive_timeout}"
         use_tool_communication="${use_tool_communication}"
         tool_voltage="${tool_voltage}"
