Commit message: dual cell mostly working

File: inspection_cell_description/urdf/inspection_cell_beta.urdf.xacro (robot description, xacro)
@@ -527,5 +527,5 @@
       <parent link="${tf_prefix}turntable_base_link"/>
       <child link="${tf_prefix}ur5e_mount_link"/>
-      <origin xyz="0 0.75 0" rpy="0 0 0"/>
+      <origin xyz="0 0.5 0" rpy="0 0 0"/>
     </joint>
     <!-- UR5e Base - Mounted on mount block -->

Commit message: new beta positions and limits

File: inspection_cell_description/urdf/inspection_cell_beta.urdf.xacro (robot description, xacro)
@@ -527,5 +527,5 @@
       <parent link="${tf_prefix}turntable_base_link"/>
       <child link="${tf_prefix}ur5e_mount_link"/>
-      <origin xyz="0 0.5 0" rpy="0 0 0"/>
+      <origin xyz="0 0.75 0" rpy="0 0 0"/>
     </joint>
     <!-- UR5e Base - Mounted on mount block -->

Commit message: beta turntable orientation change corrected.

File: inspection_cell_description/urdf/inspection_cell_beta.urdf.xacro (robot description, xacro)
@@ -516,5 +516,5 @@
       <parent link="${tf_prefix}turntable_base_link_inertia"/>
       <child link="${tf_prefix}turntable_base_link"/>
-      <origin xyz="0 0 0" rpy="0 0 0"/>
+      <origin xyz="0 0 0" rpy="0 0 ${-pi/2}"/>
     </joint>
     <joint name="${tf_prefix}ur5e_mount_to_table" type="fixed">

Commit message: added planning volume to beta, joint limit = 0.0 fix, changed the c_cpp_properties.json for macbook , settings.json for macbook - file path changed from isaac_ros-dev/

File: inspection_cell_description/urdf/inspection_cell_beta.urdf.xacro (robot description, xacro)
@@ -478,4 +478,54 @@
     <link name="${tf_prefix}turntable_base"/>
     <!-- ================================================================ -->
+    <!-- PLANNING VOLUME -->
+    <!-- ================================================================ -->
+    <!-- Define your planning volume dimensions -->
+    <xacro:property name="planning_width" value="0.620"/>   <!-- X dimension -->
+    <xacro:property name="planning_depth" value="0.620"/>   <!-- Y dimension -->
+    <xacro:property name="planning_height" value="1.000"/>  <!-- Z dimension -->
+    <xacro:property name="wall_thickness" value="0.001"/>
+    <link name="${tf_prefix}planning_volume">
+      <!-- Front wall (positive X) -->
+      <collision name="wall_front">
+      <origin xyz="${planning_width/2} 0 ${planning_height/2}" rpy="0 0 0"/>
+      <geometry>
+        <box size="${wall_thickness} ${planning_depth} ${planning_height}"/>
+      </geometry>
+      </collision>
+      <!-- Back wall (negative X) -->
+      <collision name="wall_back">
+      <origin xyz="${-planning_width/2} 0 ${planning_height/2}" rpy="0 0 0"/>
+      <geometry>
+        <box size="${wall_thickness} ${planning_depth} ${planning_height}"/>
+      </geometry>
+      </collision>
+      <!-- Left wall (positive Y) -->
+      <collision name="wall_left">
+      <origin xyz="0 ${planning_depth/2} ${planning_height/2}" rpy="0 0 0"/>
+      <geometry>
+        <box size="${planning_width} ${wall_thickness} ${planning_height}"/>
+      </geometry>
+      </collision>
+      <!-- Right wall (negative Y) -->
+      <collision name="wall_right">
+      <origin xyz="0 ${-planning_depth/2} ${planning_height/2}" rpy="0 0 0"/>
+      <geometry>
+        <box size="${planning_width} ${wall_thickness} ${planning_height}"/>
+      </geometry>
+      </collision>
+      <!-- Ceiling (positive Z) -->
+      <collision name="wall_ceiling">
+        <origin xyz="0 0 ${planning_height}" rpy="0 0 0"/>
+        <geometry>
+          <box size="${planning_width} ${planning_depth} ${wall_thickness}"/>
+        </geometry>
+      </collision>
+    </link>
+    <joint name="${tf_prefix}turntable_base_to_planning_volume" type="fixed">
+      <parent link="${tf_prefix}turntable_base_link"/>
+      <child link="${tf_prefix}planning_volume"/>
+      <origin xyz="0.0 0.325 0.0" rpy="0 0 0"/>
+    </joint>
+    <!-- ================================================================ -->
     <!-- JOINTS - OBJECT-CENTRIC UNIFIED KINEMATIC CHAIN -->
     <!-- ================================================================ -->

Commit message: changed depth camera orientation

File: inspection_cell_description/urdf/inspection_cell_beta.urdf.xacro (robot description, xacro)
@@ -25,4 +25,7 @@
   <material name="mount_black">
     <color rgba="0.1 0.1 0.1 1.0"/>
+  </material>
+  <material name="vention_blue">
+    <color rgba="0.0 0.2 0.8 1.0"/>
   </material>
   <xacro:macro name="inspection_cell" params="
@@ -756,5 +759,5 @@
       <parent link="${tf_prefix}eoat_base_link"/>
       <child link="${tf_prefix}camera_link"/>
-      <origin xyz="-0.080 0 0.06" rpy="0 ${radians(180)} 0"/>
+      <origin xyz="-0.080 0 0.06" rpy="0 0 ${radians(180)}"/>
     </joint>
     <!-- ================================================================ -->

Commit message: changed the urdf for depth camera and turntable

File: inspection_cell_description/urdf/inspection_cell_beta.urdf.xacro (robot description, xacro)
@@ -595,5 +595,5 @@
       <parent link="${tf_prefix}turntable_base_link"/>
       <child link="${tf_prefix}ur5e_mount_link"/>
-      <origin xyz="0 0.75 0" rpy="0 0 0"/>
+      <origin xyz="0 0.7287 0" rpy="0 0 0"/>
     </joint>
     <!-- UR5e Base - Mounted on mount block -->
@@ -759,5 +759,5 @@
       <parent link="${tf_prefix}eoat_base_link"/>
       <child link="${tf_prefix}camera_link"/>
-      <origin xyz="-0.080 0 0.06" rpy="${radians(180)} 0 ${radians(180)}"/>
+      <origin xyz="-0.023 0 0.033" rpy="${radians(180)} 0 ${radians(180)}"/>
     </joint>
     <!-- ================================================================ -->

Commit message: increased planning volume

File: inspection_cell_description/urdf/inspection_cell_beta.urdf.xacro (robot description, xacro)
@@ -499,6 +499,6 @@
     <!-- ================================================================ -->
     <!-- Define your planning volume dimensions -->
-    <xacro:property name="planning_width" value="0.620"/>   <!-- X dimension -->
-    <xacro:property name="planning_depth" value="0.620"/>   <!-- Y dimension -->
+    <xacro:property name="planning_width" value="1.000"/>   <!-- X dimension -->
+    <xacro:property name="planning_depth" value="1.000"/>   <!-- Y dimension -->
     <xacro:property name="planning_height" value="1.000"/>  <!-- Z dimension -->
     <xacro:property name="wall_thickness" value="0.001"/>
@@ -543,5 +543,5 @@
       <parent link="${tf_prefix}turntable_base_link"/>
       <child link="${tf_prefix}planning_volume"/>
-      <origin xyz="0.0 0.325 0.0" rpy="0 0 0"/>
+      <origin xyz="0.0 0.0 0.0" rpy="0 0 0"/>
     </joint>
     <!-- ================================================================ -->

Commit message: shortened camera

File: inspection_cell_description/urdf/inspection_cell_beta.urdf.xacro (robot description, xacro)
@@ -433,5 +433,5 @@
         <origin xyz="0 0 0.080"/>
         <geometry>
-          <cylinder radius="0.04" length="0.160"/>
+          <cylinder radius="0.04" length="0.133"/>
         </geometry>
         <material name="eoat_black"/>
@@ -440,5 +440,5 @@
         <origin xyz="0 0 0.080"/>
         <geometry>
-          <cylinder radius="0.04" length="0.160"/>
+          <cylinder radius="0.04" length="0.133"/>
         </geometry>
       </collision>

Commit message: moved camera origin

File: inspection_cell_description/urdf/inspection_cell_beta.urdf.xacro (robot description, xacro)
@@ -431,5 +431,5 @@
     <link name="${tf_prefix}eoat_camera_link">
       <visual>
-        <origin xyz="0 0 0.080"/>
+        <origin xyz="0 0 0.065"/>
         <geometry>
           <cylinder radius="0.04" length="0.133"/>
@@ -438,5 +438,5 @@
       </visual>
       <collision>
-        <origin xyz="0 0 0.080"/>
+        <origin xyz="0 0 0.065"/>
         <geometry>
           <cylinder radius="0.04" length="0.133"/>
@@ -444,5 +444,5 @@
       </collision>
       <inertial>
-        <origin xyz="0 0 0.080"/>
+        <origin xyz="0 0 0.065"/>
         <mass value="0.2"/>
         <inertia ixx="0.0002" ixy="0.0" ixz="0.0" iyy="0.0002" iyz="0.0" izz="0.0002"/>

Commit message: removed commas from beta urdf

File: inspection_cell_description/urdf/inspection_cell_beta.urdf.xacro (robot description, xacro)
@@ -453,5 +453,5 @@
         <origin xyz="0 0 0.035"/>
         <geometry>
-          <box size="0.1, 0.1 0.1"/>
+          <box size="0.1 0.1 0.1"/>
         </geometry>
         <material name="eoat_black"/>
@@ -460,5 +460,5 @@
         <origin xyz="0 0 0.0625"/>
         <geometry>
-          <box size="0.07, 0.07 0.07"/>
+          <box size="0.07 0.07 0.07"/>
         </geometry>
       </collision>

Commit message: updated camera frames

File: inspection_cell_description/urdf/inspection_cell_beta.urdf.xacro (robot description, xacro)
@@ -714,10 +714,10 @@
       <parent link="${tf_prefix}eoat_base_link"/>
       <child link="${tf_prefix}eoat_camera_link"/>
-      <origin xyz="0.024475 0 0.0475" rpy="${radians(90)} ${radians(0)} ${radians(-90)}"/>
+      <origin xyz="0.037 0 0.0365" rpy="${radians(90)} ${radians(0)} ${radians(-90)}"/>
     </joint>
     <joint name="${tf_prefix}camera_depth_optical_joint" type="fixed">
-      <parent link="${tf_prefix}eoat_base_link"/>
+      <parent link="${tf_prefix}eoat_camera_link"/>
       <child link="${tf_prefix}camera_link"/>
-      <origin xyz="-0.050287 0 -0.01232" rpy="${radians(180)} 0 ${radians(180)}"/>
+      <origin xyz="-0.009 -0.052283 0.099391" rpy="0 ${radians(-63.435)} ${radians(90)}"/>
     </joint>
     <!-- ================================================================ -->

Commit message: updated urdf and joint limits

File: inspection_cell_description/urdf/inspection_cell_beta.urdf.xacro (robot description, xacro)
@@ -699,5 +699,5 @@
       <parent link="${tf_prefix}tool0"/>
       <child link="${tf_prefix}eoat_base_link"/>
-      <origin xyz="0 0 0" rpy="0 0 ${radians(90)}"/>
+      <origin xyz="0 0 0" rpy="0 0 ${radians(-90)}"/>
     </joint>
     <joint name="${tf_prefix}eoat_top_joint" type="fixed">

Commit message: fixing joint limits and servo issues

File: inspection_cell_description/urdf/inspection_cell_beta.urdf.xacro (robot description, xacro)
@@ -699,5 +699,5 @@
       <parent link="${tf_prefix}tool0"/>
       <child link="${tf_prefix}eoat_base_link"/>
-      <origin xyz="0 0 0" rpy="0 0 ${radians(-90)}"/>
+      <origin xyz="0 0 0" rpy="0 0 ${radians(90)}"/>
     </joint>
     <joint name="${tf_prefix}eoat_top_joint" type="fixed">
@@ -716,8 +716,13 @@
       <origin xyz="0.037 0 0.0365" rpy="${radians(90)} ${radians(0)} ${radians(-90)}"/>
     </joint>
+    <!-- <joint name="${tf_prefix}camera_depth_optical_joint" type="fixed">
+      <parent link="${tf_prefix}eoat_camera_link"/>
+      <child link="${tf_prefix}camera_link"/>
+      <origin xyz="-0.09 -0.052283 0.099391" rpy="0 ${radians(-63.435)} ${radians(90)}"/>
+    </joint> -->
     <joint name="${tf_prefix}camera_depth_optical_joint" type="fixed">
       <parent link="${tf_prefix}eoat_camera_link"/>
       <child link="${tf_prefix}camera_link"/>
-      <origin xyz="-0.009 -0.052283 0.099391" rpy="0 ${radians(-63.435)} ${radians(90)}"/>
+      <origin xyz="-0.0805 0.009 0.0984" rpy="${radians(90)} ${radians(-63.435)} ${radians(0)}"/>
     </joint>
     <!-- ================================================================ -->

Commit message: Added eoat

File: inspection_cell_description/urdf/inspection_cell_beta.urdf.xacro (robot description, xacro)
@@ -390,17 +390,4 @@
     <!-- ================================================================ -->
     <link name="${tf_prefix}eoat_base_link">
-      <visual>
-        <origin xyz="0 0 0.024535"/>
-        <geometry>
-          <cylinder radius="0.0325" length="0.04907"/>
-        </geometry>
-        <material name="eoat_blue"/>
-      </visual>
-      <collision>
-        <origin xyz="0 0 0.024535"/>
-        <geometry>
-          <cylinder radius="0.0325" length="0.04907"/>
-        </geometry>
-      </collision>
       <inertial>
         <origin xyz="0 0 0.024535"/>
@@ -409,36 +396,15 @@
       </inertial>
     </link>
-    <link name="${tf_prefix}eoat_top_link">
-      <visual>
-        <origin xyz="0 0 0.024535"/>
-        <geometry>
-          <cylinder radius="0.035" length="0.001"/>
-        </geometry>
-        <material name="eoat_black"/>
-      </visual>
-      <collision>
-        <origin xyz="0 0 0.024535"/>
-        <geometry>
-          <cylinder radius="0.035" length="0.04907"/>
-        </geometry>
-      </collision>
-      <inertial>
-        <origin xyz="0 0 0.024535"/>
-        <mass value="0.05"/>
-        <inertia ixx="0.00005" ixy="0.0" ixz="0.0" iyy="0.00005" iyz="0.0" izz="0.00005"/>
-      </inertial>
-    </link>
     <link name="${tf_prefix}eoat_camera_link">
       <visual>
-        <origin xyz="0 0 0.065"/>
-        <geometry>
-          <cylinder radius="0.04" length="0.133"/>
-        </geometry>
-        <material name="eoat_black"/>
-      </visual>
-      <collision>
-        <origin xyz="0 0 0.065"/>
-        <geometry>
-          <cylinder radius="0.04" length="0.133"/>
+        <origin xyz="0 0 0" rpy="${-pi/2} 0 0"/>
+        <geometry>
+          <mesh filename="package://inspection_cell_description/meshes/visual/eoat.dae" scale="0.001 0.001 0.001"/>
+        </geometry>
+      </visual>
+      <collision>
+        <origin xyz="0 0 0" rpy="${-pi/2} 0 0"/>
+        <geometry>
+          <mesh filename="package://inspection_cell_description/meshes/collision/eoat.stl" scale="0.001 0.001 0.001"/>
         </geometry>
       </collision>
@@ -447,24 +413,4 @@
         <mass value="0.2"/>
         <inertia ixx="0.0002" ixy="0.0" ixz="0.0" iyy="0.0002" iyz="0.0" izz="0.0002"/>
-      </inertial>
-    </link>
-    <link name="${tf_prefix}eoat_body_link">
-      <visual>
-        <origin xyz="0 0 0.035"/>
-        <geometry>
-          <box size="0.1 0.1 0.1"/>
-        </geometry>
-        <material name="eoat_black"/>
-      </visual>
-      <collision>
-        <origin xyz="0 0 0.0625"/>
-        <geometry>
-          <box size="0.07 0.07 0.07"/>
-        </geometry>
-      </collision>
-      <inertial>
-        <origin xyz="0 0 0.0625"/>
-        <mass value="0.15"/>
-        <inertia ixx="0.00015" ixy="0.0" ixz="0.0" iyy="0.00015" iyz="0.0" izz="0.00015"/>
       </inertial>
     </link>
@@ -701,14 +647,4 @@
       <origin xyz="0 0 0" rpy="0 0 ${radians(90)}"/>
     </joint>
-    <joint name="${tf_prefix}eoat_top_joint" type="fixed">
-      <parent link="${tf_prefix}eoat_base_link"/>
-      <child link="${tf_prefix}eoat_top_link"/>
-      <origin xyz="0 0 0.0" rpy="0 0 0"/>
-    </joint>
-    <joint name="${tf_prefix}eoat_body_joint" type="fixed">
-      <parent link="${tf_prefix}eoat_base_link"/>
-      <child link="${tf_prefix}eoat_body_link"/>
-      <origin xyz="0.050 0 0.0475" rpy="${radians(90)} ${radians(180)} ${radians(-90)}"/>
-    </joint>
     <joint name="${tf_prefix}eoat_camera_joint" type="fixed">
       <parent link="${tf_prefix}eoat_base_link"/>

File: inspection_cell_moveit_config/config/inspection_cell.srdf.xacro (robot description, xacro)
@@ -68,22 +68,11 @@
     <disable_collisions link1="base_link_inertia" link2="turntable_disc_link" reason="Never"/>
     <disable_collisions link1="base_link_inertia" link2="ur5e_mount_link" reason="Adjacent"/>
-    <disable_collisions link1="eoat_base_link" link2="eoat_body_link" reason="Adjacent"/>
     <disable_collisions link1="eoat_base_link" link2="eoat_camera_link" reason="Adjacent"/>
-    <disable_collisions link1="eoat_base_link" link2="eoat_top_link" reason="Adjacent"/>
     <disable_collisions link1="eoat_base_link" link2="wrist_1_link" reason="Never"/>
     <disable_collisions link1="eoat_base_link" link2="wrist_2_link" reason="Never"/>
     <disable_collisions link1="eoat_base_link" link2="wrist_3_link" reason="Adjacent"/>
-    <disable_collisions link1="eoat_body_link" link2="eoat_camera_link" reason="Default"/>
-    <disable_collisions link1="eoat_body_link" link2="eoat_top_link" reason="Default"/>
-    <disable_collisions link1="eoat_body_link" link2="wrist_1_link" reason="Never"/>
-    <disable_collisions link1="eoat_body_link" link2="wrist_2_link" reason="Never"/>
-    <disable_collisions link1="eoat_body_link" link2="wrist_3_link" reason="Never"/>
-    <disable_collisions link1="eoat_camera_link" link2="eoat_top_link" reason="Default"/>
     <disable_collisions link1="eoat_camera_link" link2="wrist_1_link" reason="Never"/>
     <disable_collisions link1="eoat_camera_link" link2="wrist_2_link" reason="Never"/>
-    <disable_collisions link1="eoat_camera_link" link2="wrist_3_link" reason="Never"/>
-    <disable_collisions link1="eoat_top_link" link2="wrist_1_link" reason="Never"/>
-    <disable_collisions link1="eoat_top_link" link2="wrist_2_link" reason="Never"/>
-    <disable_collisions link1="eoat_top_link" link2="wrist_3_link" reason="Never"/>
+    <disable_collisions link1="eoat_camera_link" link2="wrist_3_link" reason="Adjacent"/>
     <disable_collisions link1="forearm_link" link2="turntable_base_link_inertia" reason="Never"/>
     <disable_collisions link1="forearm_link" link2="turntable_disc_link" reason="Never"/>

Commit message: joint limit stuff

File: inspection_cell_description/urdf/inspection_cell_beta.urdf.xacro (robot description, xacro)
@@ -123,10 +123,10 @@
     <!-- Table Link - Static visualization reference -->
     <link name="${tf_prefix}table_link">
-      <visual>
+      <!-- <visual>
         <origin xyz="0 0 0" rpy="0 0 0"/>
         <geometry>
           <mesh filename="package://inspection_cell_description/meshes/visual/table.dae"/>
         </geometry>
-      </visual>
+      </visual> -->
       <collision>
         <origin xyz="1.2192 0.762 -0.4515" rpy="0 0 0"/>
@@ -418,10 +418,10 @@
     </link>
     <link name="${tf_prefix}camera_link">
-      <visual>
+      <!-- <visual>
         <origin xyz="0 0 0" rpy="0 ${radians(90)} 0"/>
         <geometry>
           <cylinder radius="0.015" length="0.030"/>
         </geometry>
-      </visual>
+      </visual> -->
       <!-- <collision>
         <origin xyz="0 0 0" rpy="0 ${radians(90)} 0"/>
