Commit message: removed virtual link

File: inspection_cell_description/urdf/inspection_cell_beta.urdf.xacro (robot description, xacro)
@@ -189,14 +189,14 @@
     <link name="${tf_prefix}ur5e_mount_link">
       <visual>
-        <origin xyz="0 0 0.05715" rpy="0 0 0"/>
-        <geometry>
-          <box size="0.1778 0.1778 0.1143"/>
+        <origin xyz="0 0 0.03375" rpy="0 0 0"/>
+        <geometry>
+          <box size="0.1778 0.1778 0.0675"/>
         </geometry>
         <material name="mount_black"/>
       </visual>
       <collision>
-        <origin xyz="0 0 0.05715" rpy="0 0 0"/>
-        <geometry>
-          <box size="0.1778 0.1778 0.1143"/>
+        <origin xyz="0 0 0.03375" rpy="0 0 0"/>
+        <geometry>
+          <box size="0.1778 0.1778 0.0675"/>
         </geometry>
       </collision>
@@ -511,5 +511,5 @@
       <parent link="${tf_prefix}ur5e_mount_link"/>
       <child link="${tf_prefix}ur_base_link"/>
-      <origin xyz="0 0 0.0693" rpy="0 0 ${pi/2}"/>
+      <origin xyz="0 0 0.0675" rpy="0 0 ${pi/2}"/>
     </joint>
     <!-- UR Coordinate System Alignment -->

File: inspection_cell_moveit_config/config/inspection_cell.srdf.xacro (robot description, xacro)
@@ -10,14 +10,4 @@
     <!--CHAINS: When a chain is specified, all the links along the chain (including endpoints) are included in the group. Additionally, all the joints that are parents to included links are also included. This means that joints along the chain and the parent joint of the base link are included in the group-->
     <!--SUBGROUPS: Groups can also be formed by referencing to already defined group names-->
-    <!--VIRTUAL JOINT, SPIKE (Phase B): object_frame stays the URDF's actual
-    root link (object_to_disc, object_frame to turntable_disc_link, is
-    still an ordinary fixed URDF joint, unchanged) so every existing
-    consumer keyed on the link name "object_frame" (planning-scene
-    attachment, this file's own disc_to_ur5e chain base_link, orientation
-    control's live TF lookups) keeps working untouched. "root" is a new,
-    external, not-a-URDF-link frame that exists only as this virtual
-    joint's parent; a runtime-sourced (TF) correction lands here instead,
-    the same pattern as a mobile-base map-to-base_link virtual joint. -->
-    <virtual_joint name="root_to_object" type="floating" parent_frame="root" child_link="object_frame"/>
     <group name="disc_to_ur5e">
         <joint name="object_to_disc"/>
